File: Q916.kicad_sch (KiCad schematic)
At the start: 6 parts, among them J1 GPIO, U1 CAT24C256

Commit message: 初版
Parts:
- added SW1: LIMIT_SW, symbol Switch:SW_Reed
- added SW2: STOP_SW, symbol Switch:SW_Reed
- added SW3: END_BUTTON, symbol Switch:SW_Push
- added SW4: START_BUTTON, symbol Switch:SW_Push
Connections:
- net +3V3: now also SW1.2, SW2.2, SW3.2
- net GND: now also SW4.2
- net GPIO[10]/SPI0.MOSI: now also SW3.1
- net GPIO[23]: now also SW1.1
- net GPIO[9]/SPI0.MISO: now also SW4.1
Other:
- title: (none) -> Monorail Camera
Changed lines of the file:
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@@
   (paper "A4")
   (title_block
+    (title "Monorail Camera")
     (date "15 nov 2012")
+    (rev "1.00")
   )
   (junction (at 93.98 175.26) (diameter 1.016) (color 0 0 0 0)
@@
   (junction (at 81.28 165.1) (diameter 1.016) (color 0 0 0 0)
   )
+  (junction (at 154.94 63.5) (diameter 0) (color 0 0 0 0)
+  )
   (junction (at 101.6 165.1) (diameter 1.016) (color 0 0 0 0)
   )
@@
   )
   (junction (at 76.2 63.5) (diameter 1.016) (color 0 0 0 0)
+  )
+  (junction (at 154.94 76.2) (diameter 0) (color 0 0 0 0)
   )
   (junction (at 76.2 50.8) (diameter 1.016) (color 0 0 0 0)
@@
   (no_connect (at 71.12 177.8))
   (no_connect (at 71.12 180.34))
+  (wire (pts (xy 149.86 63.5) (xy 154.94 63.5))
+    (stroke (width 0) (type default) (color 0 0 0 0))
+  )
   (wire (pts (xy 58.42 58.42) (xy 58.42 76.2))
     (stroke (width 0) (type solid) (color 0 0 0 0))
@@
     (stroke (width 0) (type solid) (color 0 0 0 0))
   )
+  (wire (pts (xy 149.86 76.2) (xy 154.94 76.2))
+    (stroke (width 0) (type default) (color 0 0 0 0))
+  )
   (wire (pts (xy 58.42 38.1) (xy 60.96 38.1))
     (stroke (width 0) (type solid) (color 0 0 0 0))
@@
     (stroke (width 0) (type solid) (color 0 0 0 0))
   )
+  (wire (pts (xy 24.13 88.9) (xy 139.7 88.9))
+    (stroke (width 0) (type default) (color 0 0 0 0))
+  )
   (wire (pts (xy 73.66 55.88) (xy 100.33 55.88))
     (stroke (width 0) (type solid) (color 0 0 0 0))
@@
     (stroke (width 0) (type solid) (color 0 0 0 0))
   )
+  (wire (pts (xy 25.4 101.6) (xy 139.7 101.6))
+    (stroke (width 0) (type default) (color 0 0 0 0))
+  )
   (wire (pts (xy 58.42 58.42) (xy 60.96 58.42))
     (stroke (width 0) (type solid) (color 0 0 0 0))
@@
     (stroke (width 0) (type solid) (color 0 0 0 0))
   )
-  (wire (pts (xy 73.66 45.72) (xy 100.33 45.72))
+  (wire (pts (xy 73.66 45.72) (xy 133.35 45.72))
     (stroke (width 0) (type solid) (color 0 0 0 0))
   )
@@
     (stroke (width 0) (type solid) (color 0 0 0 0))
   )
+  (wire (pts (xy 133.35 63.5) (xy 139.7 63.5))
+    (stroke (width 0) (type default) (color 0 0 0 0))
+  )
   (wire (pts (xy 73.66 76.2) (xy 100.33 76.2))
     (stroke (width 0) (type solid) (color 0 0 0 0))
@@
     (stroke (width 0) (type solid) (color 0 0 0 0))
   )
+  (wire (pts (xy 133.35 45.72) (xy 133.35 63.5))
+    (stroke (width 0) (type default) (color 0 0 0 0))
+  )
   (wire (pts (xy 76.2 68.58) (xy 73.66 68.58))
     (stroke (width 0) (type solid) (color 0 0 0 0))
@@
     (stroke (width 0) (type solid) (color 0 0 0 0))
   )
+  (wire (pts (xy 154.94 88.9) (xy 149.86 88.9))
+    (stroke (width 0) (type default) (color 0 0 0 0))
+  )
   (wire (pts (xy 60.96 30.48) (xy 31.75 30.48))
     (stroke (width 0) (type solid) (color 0 0 0 0))
@@
     (stroke (width 0) (type solid) (color 0 0 0 0))
   )
+  (wire (pts (xy 25.4 53.34) (xy 25.4 101.6))
+    (stroke (width 0) (type default) (color 0 0 0 0))
+  )
   (wire (pts (xy 76.2 43.18) (xy 76.2 50.8))
     (stroke (width 0) (type solid) (color 0 0 0 0))
@@
     (stroke (width 0) (type solid) (color 0 0 0 0))
   )
+  (wire (pts (xy 154.94 63.5) (xy 154.94 76.2))
+    (stroke (width 0) (type default) (color 0 0 0 0))
+  )
   (wire (pts (xy 31.75 45.72) (xy 60.96 45.72))
     (stroke (width 0) (type solid) (color 0 0 0 0))
   )
-  (wire (pts (xy 31.75 53.34) (xy 60.96 53.34))
-    (stroke (width 0) (type solid) (color 0 0 0 0))
+  (wire (pts (xy 25.4 53.34) (xy 60.96 53.34))
+    (stroke (width 0) (type solid) (color 0 0 0 0))
+  )
+  (wire (pts (xy 24.13 50.8) (xy 24.13 88.9))
+    (stroke (width 0) (type default) (color 0 0 0 0))
   )
   (wire (pts (xy 31.75 66.04) (xy 60.96 66.04))
@@
     (stroke (width 0) (type solid) (color 0 0 0 0))
   )
+  (wire (pts (xy 154.94 76.2) (xy 154.94 88.9))
+    (stroke (width 0) (type default) (color 0 0 0 0))
+  )
   (wire (pts (xy 31.75 71.12) (xy 60.96 71.12))
     (stroke (width 0) (type solid) (color 0 0 0 0))
@@
     (stroke (width 0) (type solid) (color 0 0 0 0))
   )
+  (wire (pts (xy 149.86 101.6) (xy 153.67 101.6))
+    (stroke (width 0) (type default) (color 0 0 0 0))
+  )
   (wire (pts (xy 76.2 68.58) (xy 76.2 80.01))
     (stroke (width 0) (type solid) (color 0 0 0 0))
@@
     (stroke (width 0) (type solid) (color 0 0 0 0))
   )
-  (wire (pts (xy 60.96 50.8) (xy 31.75 50.8))
+  (wire (pts (xy 154.94 50.8) (xy 154.94 63.5))
+    (stroke (width 0) (type default) (color 0 0 0 0))
+  )
+  (wire (pts (xy 24.13 50.8) (xy 60.96 50.8))
     (stroke (width 0) (type solid) (color 0 0 0 0))
   )
   (wire (pts (xy 73.66 60.96) (xy 100.33 60.96))
     (stroke (width 0) (type solid) (color 0 0 0 0))
+  )
+  (wire (pts (xy 153.67 101.6) (xy 153.67 104.14))
+    (stroke (width 0) (type default) (color 0 0 0 0))
   )
   (text "Additional pin functions:\nhttps://pinout.xyz/" (at 179.07 180.34 0)
@@
     (pin "2")
   )
+  (symbol (lib_id "Switch:SW_Reed") (at 144.78 76.2 0) (unit 1)
+    (in_bom yes) (on_board yes) (fields_autoplaced)
+    (property "Reference" "SW2" (id 0) (at 144.78 71.1032 0))
+    (property "Value" "STOP_SW" (id 1) (at 144.78 73.6401 0))
+    (property "Footprint" "" (id 2) (at 144.78 76.2 0)
+      (effects (font (size 1.27 1.27)) hide)
+    )
+    (property "Datasheet" "~" (id 3) (at 144.78 76.2 0)
+      (effects (font (size 1.27 1.27)) hide)
+    )
+    (pin "1")
+    (pin "2")
+  )
   (symbol (lib_id "Device:R_Small") (at 101.6 170.18 0) (unit 1)
     (in_bom yes) (on_board yes)
@@
     )
     (pin "1")
+  )
+  (symbol (lib_id "Switch:SW_Reed") (at 144.78 63.5 0) (unit 1)
+    (in_bom yes) (on_board yes) (fields_autoplaced)
+    (property "Reference" "SW1" (id 0) (at 144.78 58.4032 0))
+    (property "Value" "LIMIT_SW" (id 1) (at 144.78 60.9401 0))
+    (property "Footprint" "" (id 2) (at 144.78 63.5 0)
+      (effects (font (size 1.27 1.27)) hide)
+    )
+    (property "Datasheet" "~" (id 3) (at 144.78 63.5 0)
+      (effects (font (size 1.27 1.27)) hide)
+    )
+    (pin "1")
+    (pin "2")
   )
   (symbol (lib_id "Memory_EEPROM:CAT24C256") (at 81.28 177.8 0) (unit 1)
@@
     (pin "8")
   )
+  (symbol (lib_id "Switch:SW_Push") (at 144.78 101.6 0) (unit 1)
+    (in_bom yes) (on_board yes) (fields_autoplaced)
+    (property "Reference" "SW4" (id 0) (at 144.78 94.9792 0))
+    (property "Value" "START_BUTTON" (id 1) (at 144.78 97.5161 0))
+    (property "Footprint" "" (id 2) (at 144.78 96.52 0)
+      (effects (font (size 1.27 1.27)) hide)
+    )
+    (property "Datasheet" "~" (id 3) (at 144.78 96.52 0)
+      (effects (font (size 1.27 1.27)) hide)
+    )
+    (pin "1")
+    (pin "2")
+  )
+  (symbol (lib_id "power:+3.3V") (at 154.94 50.8 0) (unit 1)
+    (in_bom yes) (on_board yes)
+    (property "Reference" "#PWR?" (id 0) (at 154.94 54.61 0)
+      (effects (font (size 1.27 1.27)) hide)
+    )
+    (property "Value" "+3.3V" (id 1) (at 155.3083 46.4756 0))
+    (property "Footprint" "" (id 2) (at 154.94 50.8 0))
+    (property "Datasheet" "" (id 3) (at 154.94 50.8 0))
+    (pin "1")
+  )
+  (symbol (lib_id "Switch:SW_Push") (at 144.78 88.9 0) (unit 1)
+    (in_bom yes) (on_board yes) (fields_autoplaced)
+    (property "Reference" "SW3" (id 0) (at 144.78 82.2792 0))
+    (property "Value" "END_BUTTON" (id 1) (at 144.78 84.8161 0))
+    (property "Footprint" "" (id 2) (at 144.78 83.82 0)
+      (effects (font (size 1.27 1.27)) hide)
+    )
+    (property "Datasheet" "~" (id 3) (at 144.78 83.82 0)
+      (effects (font (size 1.27 1.27)) hide)
+    )
+    (pin "1")
+    (pin "2")
+  )
   (symbol (lib_id "power:GND") (at 81.28 190.5 0) (unit 1)
     (in_bom yes) (on_board yes)
@@
     (pin "1")
   )
+  (symbol (lib_id "power:GND") (at 153.67 104.14 0) (unit 1)
+    (in_bom yes) (on_board yes)
+    (property "Reference" "#PWR?" (id 0) (at 153.67 110.49 0)
+      (effects (font (size 1.27 1.27)) hide)
+    )
+    (property "Value" "GND" (id 1) (at 153.7843 108.4644 0))
+    (property "Footprint" "" (id 2) (at 153.67 104.14 0))
+    (property "Datasheet" "" (id 3) (at 153.67 104.14 0))
+    (pin "1")
+  )
   (symbol (lib_id "power:+3.3V") (at 101.6 180.34 270) (unit 1)
     (in_bom yes) (on_board yes)
@@
       (reference "#PWR0103") (unit 1) (value "+3.3V") (footprint "")
     )
+    (path "/91badf57-9205-41b3-868e-d2f76a8d3568"
+      (reference "#PWR?") (unit 1) (value "+3.3V") (footprint "")
+    )
+    (path "/cebcecf5-87ae-4508-8ffc-93cda567aff6"
+      (reference "#PWR?") (unit 1) (value "GND") (footprint "")
+    )
     (path "/0f7872a7-de47-41d5-a21f-9934102d3a5f"
       (reference "C1") (unit 1) (value "100n") (footprint "")
@@
       (reference "R2") (unit 1) (value "3.9k") (footprint "")
     )
+    (path "/6d585646-5909-4295-86b9-92b258f35ac1"
+      (reference "SW1") (unit 1) (value "LIMIT_SW") (footprint "")
+    )
+    (path "/4a7edba3-3d68-4c19-93f5-bcacc18e7f3d"
+      (reference "SW2") (unit 1) (value "STOP_SW") (footprint "")
+    )
+    (path "/b02b8a1b-a036-4d1d-b440-172a8cf842a3"
+      (reference "SW3") (unit 1) (value "END_BUTTON") (footprint "")
+    )
+    (path "/706bc8e1-cc29-46e0-98f9-fbbe941cb3e0"
+      (reference "SW4") (unit 1) (value "START_BUTTON") (footprint "")
+    )
     (path "/6d6e5c8e-c0cf-4e61-9c00-723a754d58be"
